File: Element14_AudioServo.sch (EAGLE design)
At the start: 0 parts

Commit message: Update Element14_AudioServo.sch
Other:
- note added: "GND"
- note added: "POWER +5V"
- note added: "SIGNAL"
- note added: "TO SERVO"
Changed lines of the file:
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@@
 <setting verticaltext="up"/>
 </settings>
-<grid distance="0.1" unitdist="inch" unit="inch" style="lines" multiple="1" display="no" altdistance="0.01" altunitdist="inch" altunit="inch"/>
+<grid distance="0.1" unitdist="inch" unit="inch" style="lines" multiple="1" display="yes" altdistance="0.01" altunitdist="inch" altunit="inch"/>
 <layers>
 <layer number="1" name="Top" color="4" fill="1" visible="no" active="no"/>
@@
 </variantdefs>
 <parts>
+<part name="IC1" library="st-microelectronics" deviceset="NE555" device=""/>
+<part name="R1" library="resistor" deviceset="R-US_" device="R0805" value="220k"/>
+<part name="R2" library="resistor" deviceset="R-US_" device="R0805" value="4.7k"/>
+<part name="R3" library="resistor" deviceset="R-US_" device="R0805" value="10k"/>
+<part name="R4" library="resistor" deviceset="R-US_" device="R0805" value="10k"/>
+<part name="C1" library="resistor" deviceset="C-US" device="C0805" value="0.01uF"/>
+<part name="GND1" library="supply1" deviceset="GND" device=""/>
+<part name="GND2" library="supply1" deviceset="GND" device=""/>
+<part name="GND3" library="supply1" deviceset="GND" device=""/>
+<part name="C2" library="resistor" deviceset="C-US" device="C0805" value="0.1uF"/>
+<part name="T1" library="transistor" deviceset="*-NPN-" device="SOT23-EBC"/>
+<part name="GND4" library="supply1" deviceset="GND" device=""/>
+<part name="R6" library="murata-potentiometer" deviceset="PVG3" device="" value="50k"/>
+<part name="C3" library="resistor" deviceset="C-US" device="C0805" value="470uF"/>
+<part name="GND5" library="supply1" deviceset="GND" device=""/>
 </parts>
 <sheets>
 <sheet>
 <plain>
+<text x="134.62" y="58.42" size="1.778" layer="91">TO SERVO</text>
+<text x="137.16" y="53.34" size="1.778" layer="91">SIGNAL</text>
+<text x="137.16" y="43.18" size="1.778" layer="91">POWER +5V</text>
+<text x="139.7" y="27.94" size="1.778" layer="91">GND</text>
 </plain>
 <instances>
+<instance part="IC1" gate="G$1" x="76.2" y="48.26"/>
+<instance part="R1" gate="G$1" x="45.72" y="63.5" rot="R90"/>
+<instance part="R2" gate="G$1" x="45.72" y="33.02" rot="R90"/>
+<instance part="R3" gate="G$1" x="99.06" y="48.26" rot="R180"/>
+<instance part="R4" gate="G$1" x="114.3" y="63.5" rot="R270"/>
+<instance part="C1" gate="G$1" x="96.52" y="35.56"/>
+<instance part="GND1" gate="1" x="96.52" y="27.94"/>
+<instance part="GND2" gate="1" x="91.44" y="27.94"/>
+<instance part="GND3" gate="1" x="60.96" y="12.7"/>
+<instance part="C2" gate="G$1" x="60.96" y="20.32"/>
+<instance part="T1" gate="G$1" x="111.76" y="48.26"/>
+<instance part="GND4" gate="1" x="114.3" y="27.94"/>
+<instance part="R6" gate="G$1" x="53.34" y="40.64" rot="R90"/>
+<instance part="C3" gate="G$1" x="127" y="38.1"/>
+<instance part="GND5" gate="1" x="127" y="27.94"/>
 </instances>
 <busses>
 </busses>
 <nets>
+<net name="N$1" class="0">
+<segment>
+<pinref part="IC1" gate="G$1" pin="CON"/>
+<pinref part="C1" gate="G$1" pin="1"/>
+<wire x1="86.36" y1="43.18" x2="96.52" y2="43.18" width="0.1524" layer="91"/>
+<wire x1="96.52" y1="43.18" x2="96.52" y2="38.1" width="0.1524" layer="91"/>
+</segment>
+</net>
+<net name="GND" class="0">
+<segment>
+<pinref part="C1" gate="G$1" pin="2"/>
+<pinref part="GND1" gate="1" pin="GND"/>
+</segment>
+<segment>
+<pinref part="IC1" gate="G$1" pin="GND"/>
+<wire x1="86.36" y1="40.64" x2="91.44" y2="40.64" width="0.1524" layer="91"/>
+<wire x1="91.44" y1="40.64" x2="91.44" y2="30.48" width="0.1524" layer="91"/>
+<pinref part="GND2" gate="1" pin="GND"/>
+</segment>
+<segment>
+<pinref part="GND3" gate="1" pin="GND"/>
+<pinref part="C2" gate="G$1" pin="2"/>
+</segment>
+<segment>
+<pinref part="T1" gate="G$1" pin="E"/>
+<pinref part="GND4" gate="1" pin="GND"/>
+<wire x1="114.3" y1="43.18" x2="114.3" y2="30.48" width="0.1524" layer="91"/>
+</segment>
+<segment>
+<pinref part="C3" gate="G$1" pin="2"/>
+<pinref part="GND5" gate="1" pin="GND"/>
+<wire x1="127" y1="33.02" x2="127" y2="30.48" width="0.1524" layer="91"/>
+<wire x1="127" y1="30.48" x2="144.78" y2="30.48" width="0.1524" layer="91"/>
+</segment>
+</net>
+<net name="N$3" class="0">
+<segment>
+<pinref part="IC1" gate="G$1" pin="OUT"/>
+<pinref part="R3" gate="G$1" pin="2"/>
+<wire x1="86.36" y1="48.26" x2="93.98" y2="48.26" width="0.1524" layer="91"/>
+</segment>
+</net>
+<net name="N$4" class="0">
+<segment>
+<pinref part="R3" gate="G$1" pin="1"/>
+<pinref part="T1" gate="G$1" pin="B"/>
+<wire x1="104.14" y1="48.26" x2="109.22" y2="48.26" width="0.1524" layer="91"/>
+</segment>
+</net>
+<net name="N$5" class="0">
+<segment>
+<pinref part="R4" gate="G$1" pin="2"/>
+<pinref part="T1" gate="G$1" pin="C"/>
+<wire x1="114.3" y1="58.42" x2="114.3" y2="55.88" width="0.1524" layer="91"/>
+<wire x1="114.3" y1="55.88" x2="114.3" y2="53.34" width="0.1524" layer="91"/>
+<wire x1="114.3" y1="55.88" x2="124.46" y2="55.88" width="0.1524" layer="91"/>
+<wire x1="124.46" y1="55.88" x2="124.46" y2="58.42" width="0.1524" layer="91"/>
+<wire x1="124.46" y1="58.42" x2="129.54" y2="58.42" width="0.1524" layer="91"/>
+<wire x1="129.54" y1="58.42" x2="129.54" y2="55.88" width="0.1524" layer="91"/>
+<wire x1="129.54" y1="55.88" x2="144.78" y2="55.88" width="0.1524" layer="91"/>
+<junction x="114.3" y="55.88"/>
+</segment>
+</net>
+<net name="N$6" class="0">
+<segment>
+<pinref part="IC1" gate="G$1" pin="VCC+"/>
+<wire x1="86.36" y1="55.88" x2="91.44" y2="55.88" width="0.1524" layer="91"/>
+<wire x1="91.44" y1="55.88" x2="91.44" y2="71.12" width="0.1524" layer="91"/>
+<pinref part="R4" gate="G$1" pin="1"/>
+<wire x1="91.44" y1="71.12" x2="114.3" y2="71.12" width="0.1524" layer="91"/>
+<wire x1="114.3" y1="71.12" x2="114.3" y2="68.58" width="0.1524" layer="91"/>
+<pinref part="IC1" gate="G$1" pin="/RES"/>
+<wire x1="86.36" y1="53.34" x2="91.44" y2="53.34" width="0.1524" layer="91"/>
+<wire x1="91.44" y1="53.34" x2="91.44" y2="55.88" width="0.1524" layer="91"/>
+<junction x="91.44" y="55.88"/>
+<pinref part="R1" gate="G$1" pin="2"/>
+<wire x1="91.44" y1="71.12" x2="45.72" y2="71.12" width="0.1524" layer="91"/>
+<wire x1="45.72" y1="71.12" x2="45.72" y2="68.58" width="0.1524" layer="91"/>
+<junction x="91.44" y="71.12"/>
+<pinref part="C3" gate="G$1" pin="1"/>
+<wire x1="127" y1="40.64" x2="127" y2="45.72" width="0.1524" layer="91"/>
+<wire x1="127" y1="45.72" x2="127" y2="71.12" width="0.1524" layer="91"/>
+<wire x1="127" y1="71.12" x2="114.3" y2="71.12" width="0.1524" layer="91"/>
+<junction x="114.3" y="71.12"/>
+<wire x1="127" y1="45.72" x2="144.78" y2="45.72" width="0.1524" layer="91"/>
+<junction x="127" y="45.72"/>
+</segment>
+</net>
+<net name="N$7" class="0">
+<segment>
+<pinref part="IC1" gate="G$1" pin="TRI"/>
+<wire x1="66.04" y1="40.64" x2="60.96" y2="40.64" width="0.1524" layer="91"/>
+<wire x1="60.96" y1="40.64" x2="60.96" y2="25.4" width="0.1524" layer="91"/>
+<pinref part="C2" gate="G$1" pin="1"/>
+<pinref part="IC1" gate="G$1" pin="TRE"/>
+<wire x1="60.96" y1="25.4" x2="60.96" y2="22.86" width="0.1524" layer="91"/>
+<wire x1="66.04" y1="48.26" x2="60.96" y2="48.26" width="0.1524" layer="91"/>
+<wire x1="60.96" y1="48.26" x2="60.96" y2="40.64" width="0.1524" layer="91"/>
+<junction x="60.96" y="40.64"/>
+<pinref part="R2" gate="G$1" pin="1"/>
+<wire x1="45.72" y1="27.94" x2="45.72" y2="25.4" width="0.1524" layer="91"/>
+<wire x1="45.72" y1="25.4" x2="60.96" y2="25.4" width="0.1524" layer="91"/>
+<junction x="60.96" y="25.4"/>
+</segment>
+</net>
+<net name="N$8" class="0">
+<segment>
+<pinref part="R6" gate="G$1" pin="1"/>
+<pinref part="R2" gate="G$1" pin="2"/>
+<wire x1="45.72" y1="40.64" x2="45.72" y2="38.1" width="0.1524" layer="91"/>
+</segment>
+</net>
+<net name="N$9" class="0">
+<segment>
+<pinref part="R6" gate="G$1" pin="2"/>
+<pinref part="IC1" gate="G$1" pin="DIS"/>
+<wire x1="66.04" y1="55.88" x2="45.72" y2="55.88" width="0.1524" layer="91"/>
+<wire x1="45.72" y1="55.88" x2="45.72" y2="50.8" width="0.1524" layer="91"/>
+<pinref part="R1" gate="G$1" pin="1"/>
+<wire x1="45.72" y1="58.42" x2="45.72" y2="55.88" width="0.1524" layer="91"/>
+<junction x="45.72" y="55.88"/>
+</segment>
+</net>
 </nets>
 </sheet>
@@
 <moduleinsts>
 <moduleinst name="AUDIO_AMP" module="AUDIO_AMP" x="-63.5" y="12.7"/>
-<moduleinst name="TIMER" module="TIMER" x="-63.5" y="-45.72"/>
+<moduleinst name="TIMER" module="TIMER" x="-60.96" y="-60.96"/>
 <moduleinst name="POWER" module="POWER" x="-119.38" y="-17.78"/>
 </moduleinsts>

Commit message: Update Element14_AudioServo.sch
Added HC4066 block
Changed lines of the file:
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@@
 <part name="T1" library="transistor" deviceset="*-NPN-" device="SOT23-EBC"/>
 <part name="GND4" library="supply1" deviceset="GND" device=""/>
-<part name="R6" library="murata-potentiometer" deviceset="PVG3" device="" value="50k"/>
+<part name="R6" library="El14_AudioServo" deviceset="PVG3_POTENTIOMETER" device="" value="50k"/>
 <part name="C3" library="resistor" deviceset="C-US" device="C0805" value="470uF"/>
 <part name="GND5" library="supply1" deviceset="GND" device=""/>
@@
 <pinref part="R6" gate="G$1" pin="1"/>
 <pinref part="R2" gate="G$1" pin="2"/>
-<wire x1="45.72" y1="40.64" x2="45.72" y2="38.1" width="0.1524" layer="91"/>
+<wire x1="45.72" y1="45.72" x2="45.72" y2="38.1" width="0.1524" layer="91"/>
 </segment>
 </net>
@@
 <pinref part="IC1" gate="G$1" pin="DIS"/>
 <wire x1="66.04" y1="55.88" x2="45.72" y2="55.88" width="0.1524" layer="91"/>
-<wire x1="45.72" y1="55.88" x2="45.72" y2="50.8" width="0.1524" layer="91"/>
 <pinref part="R1" gate="G$1" pin="1"/>
 <wire x1="45.72" y1="58.42" x2="45.72" y2="55.88" width="0.1524" layer="91"/>
@@
 </sheets>
 </module>
+<module name="SWITCH" prefix="" dx="30.48" dy="20.32">
+<ports>
+</ports>
+<variantdefs>
+</variantdefs>
+<parts>
+<part name="74HC4066" library="El14_AudioServo" deviceset="74HC4066" device="" value="U1"/>
+<part name="GND1" library="supply1" deviceset="GND" device=""/>
+<part name="R1" library="resistor" deviceset="R-US_" device="R0805"/>
+<part name="R2" library="resistor" deviceset="R-US_" device="R0805"/>
+<part name="R3" library="resistor" deviceset="R-US_" device="R0805"/>
+<part name="LED1" library="arduino_Uno_Rev3-02-TH" deviceset="LED" device=""/>
+<part name="GND2" library="supply1" deviceset="GND" device=""/>
+</parts>
+<sheets>
+<sheet>
+<plain>
+</plain>
+<instances>
+<instance part="74HC4066" gate="G$1" x="12.7" y="7.62"/>
+<instance part="GND1" gate="1" x="50.8" y="0"/>
+<instance part="R1" gate="G$1" x="-20.32" y="5.08"/>
+<instance part="R2" gate="G$1" x="-5.08" y="-7.62" rot="R90"/>
+<instance part="R3" gate="G$1" x="-15.24" y="30.48" rot="R180"/>
+<instance part="LED1" gate="G$1" x="-2.54" y="30.48" rot="R90"/>
+<instance part="GND2" gate="1" x="-5.08" y="-20.32"/>
+</instances>
+<busses>
+</busses>
+<nets>
+<net name="GND" class="0">
+<segment>
+<pinref part="74HC4066" gate="G$1" pin="1B"/>
+<wire x1="38.1" y1="35.56" x2="50.8" y2="35.56" width="0.1524" layer="91"/>
+<pinref part="GND1" gate="1" pin="GND"/>
+<wire x1="50.8" y1="35.56" x2="50.8" y2="30.48" width="0.1524" layer="91"/>
+<pinref part="74HC4066" gate="G$1" pin="2C"/>
+<wire x1="50.8" y1="30.48" x2="50.8" y2="25.4" width="0.1524" layer="91"/>
+<wire x1="50.8" y1="25.4" x2="50.8" y2="20.32" width="0.1524" layer="91"/>
+<wire x1="50.8" y1="20.32" x2="50.8" y2="2.54" width="0.1524" layer="91"/>
+<wire x1="38.1" y1="30.48" x2="50.8" y2="30.48" width="0.1524" layer="91"/>
+<pinref part="74HC4066" gate="G$1" pin="3C"/>
+<wire x1="38.1" y1="25.4" x2="50.8" y2="25.4" width="0.1524" layer="91"/>
+<pinref part="74HC4066" gate="G$1" pin="GND"/>
+<wire x1="38.1" y1="20.32" x2="50.8" y2="20.32" width="0.1524" layer="91"/>
+<junction x="50.8" y="20.32"/>
+<junction x="50.8" y="25.4"/>
+<junction x="50.8" y="30.48"/>
+</segment>
+<segment>
+<pinref part="R2" gate="G$1" pin="1"/>
+<pinref part="GND2" gate="1" pin="GND"/>
+<wire x1="-5.08" y1="-12.7" x2="-5.08" y2="-17.78" width="0.1524" layer="91"/>
+</segment>
+</net>
+<net name="N$2" class="0">
+<segment>
+<pinref part="74HC4066" gate="G$1" pin="1C"/>
+<wire x1="10.16" y1="10.16" x2="5.08" y2="10.16" width="0.1524" layer="91"/>
+<wire x1="5.08" y1="10.16" x2="5.08" y2="5.08" width="0.1524" layer="91"/>
+<pinref part="74HC4066" gate="G$1" pin="4C"/>
+<wire x1="5.08" y1="5.08" x2="10.16" y2="5.08" width="0.1524" layer="91"/>
+<pinref part="R1" gate="G$1" pin="2"/>
+<wire x1="5.08" y1="5.08" x2="-5.08" y2="5.08" width="0.1524" layer="91"/>
+<pinref part="R2" gate="G$1" pin="2"/>
+<wire x1="-5.08" y1="5.08" x2="-15.24" y2="5.08" width="0.1524" layer="91"/>
+<wire x1="-5.08" y1="-2.54" x2="-5.08" y2="5.08" width="0.1524" layer="91"/>
+<junction x="-5.08" y="5.08"/>
+<junction x="5.08" y="5.08"/>
+</segment>
+</net>
+<net name="N$3" class="0">
+<segment>
+<pinref part="74HC4066" gate="G$1" pin="1A"/>
+<pinref part="LED1" gate="G$1" pin="C"/>
+<wire x1="10.16" y1="30.48" x2="2.54" y2="30.48" width="0.1524" layer="91"/>
+</segment>
+</net>
+<net name="N$4" class="0">
+<segment>
+<pinref part="LED1" gate="G$1" pin="A"/>
+<pinref part="R3" gate="G$1" pin="1"/>
+<wire x1="-5.08" y1="30.48" x2="-10.16" y2="30.48" width="0.1524" layer="91"/>
+</segment>
+</net>
+<net name="N$5" class="0">
+<segment>
+<pinref part="R3" gate="G$1" pin="2"/>
+<wire x1="-20.32" y1="30.48" x2="-22.86" y2="30.48" width="0.1524" layer="91"/>
+<wire x1="-22.86" y1="30.48" x2="-22.86" y2="35.56" width="0.1524" layer="91"/>
+<pinref part="74HC4066" gate="G$1" pin="VCC"/>
+<wire x1="-22.86" y1="35.56" x2="10.16" y2="35.56" width="0.1524" layer="91"/>
+</segment>
+</net>
+</nets>
+</sheet>
+</sheets>
+</module>
 </modules>
 <parts>
@@
 <moduleinst name="TIMER" module="TIMER" x="-60.96" y="-60.96"/>
 <moduleinst name="POWER" module="POWER" x="-119.38" y="-17.78"/>
+<moduleinst name="SWITCH1" module="SWITCH" x="-116.84" y="-60.96"/>
 </moduleinsts>
 <instances>
