File: Element14_AudioServo.brd (EAGLE design)
At the start: 68.6 x 53.3 mm, 53 parts, among them T1 FDN340P, U1 NCP1117ST50T3G, U2 LP2985-33DBVR, U3 ATMEGA16U2-MU(R), U5 LMV358IDGKR, X1 POWERSUPPLY_DC21MMX, X2 USB-B_TH, Y1 16MHz, Y2 CSTCE16M0V53-R0 16MHZ

Commit message: put some parts in
Parts:
- removed AD: 6x1F-H8.5, SmartPrj:1X06
- removed C1, C2, C4, C5, C6, C7: 100n, SmartPrj:C0603-ROUND
- removed C11, C9: 22p, SmartPrj:C0603-ROUND
- removed C3, C8: 1u, SmartPrj:C0603-ROUND
- removed D1: M7, diode:SMB
- removed D2, D3: CD1206-S01575, diode:MINIMELF
- removed F1: MF-MSMF050-2 500mA, rcl:L1812
- removed FD1, FD2, FD3: FIDUCIALMOUNT, SmartPrj:FIDUCIA-MOUNT
- removed GROUND, RESET-EN: (no value), jumper:SJ
- removed ICSP, ICSP1: 3x2 M, SmartPrj:2X03
- removed IOH: 10x1F-H8.5, SmartPrj:1X10@1
- removed IOL, POWER: 8x1F-H8.5, SmartPrj:1X08
- removed JP2: 2x2 M - NM, SmartPrj:2X02
- removed L, RX, TX: YELLOW, led:CHIP-LED0805
- removed L1: BLM21, wuerth-elektronik:0805
- removed ON: GREEN, led:CHIP-LED0805
- removed PC1, PC2: 47u, rcl:PANASONIC_D
- removed R1, R2: 1M, SmartPrj:R0603-ROUND
- removed RESET: TS42031-160R-TR-7260, SmartPrj:TS42
- removed RN1: 10K, resistor-dil:CAY16
- removed RN2, RN4: 1K, resistor-dil:CAY16
- removed RN3: 22R, resistor-dil:CAY16
- removed T1: FDN340P, zetex:SOT-23
- removed U$1: DISCLAIMER, SmartPrj:DISCLAIMER
- removed U1: NCP1117ST50T3G, linear:SOT223
- removed U2: LP2985-33DBVR, SmartPrj:SOT23-DBV
- removed U3: ATMEGA16U2-MU(R), SmartPrj:MLF32
- removed U5: LMV358IDGKR, linear:MSOP08
- removed X1: POWERSUPPLY_DC21MMX, SmartPrj:POWERSUPPLY_DC-21MM
- removed X2: USB-B_TH, SmartPrj:PN61729
- removed Y1: 16MHz, SmartPrj:QS
- removed Y2: CSTCE16M0V53-R0 16MHZ, SmartPrj:RESONATOR
- removed Z1, Z2: CG0603MLC-05E, varistor:CT/CN0603
- removed ZU4: ATMEGA328P-PU, SmartPrj:DIL28-3
Connections:
- removed net +3V3: C3.2, POWER.4, U2.5, U5.2
- removed net +5V: C1.2, C2.2, C6.2, C7.1, D2.C, D3.C, ICSP.2, ICSP1.2, PC2.+, POWER.2, POWER.5, RN1.3, RN1.5, RN2.2, RN2.3, RN4.3, RN4.4, T1.2, U1.2, U1.4, U2.1, U2.3, U3.32, U3.4, U5.8, ZU4.20, ZU4.7
- removed net 5-GND: RESET.5
- removed net AD0: AD.1, ZU4.23
- removed net AD1: AD.2, ZU4.24
- removed net AD2: AD.3, ZU4.25
- removed net AD3: AD.4, ZU4.26
- removed net AD4/SDA: AD.5, IOH.9, ZU4.27
- removed net AD5/SCL: AD.6, IOH.10, ZU4.28
- removed net AREF: C4.2, IOH.8, ZU4.21
- removed net CMP: RN1.1, RN1.2, U5.3
- removed net D+: RN3.5, X2.3, Z1.1
- removed net D-: RN3.8, X2.2, Z2.1
- removed net DTR: C5.1, RN2.4, U3.13
- removed net GATE_CMD: T1.3, U5.1
- removed net GND: C1.1, C11.2, C2.1, C3.1, C4.1, C6.1, C7.2, C9.2, GROUND.1, ICSP.6, ICSP1.6, IOH.7, L.C, ON.C, PC1.-, PC2.-, POWER.6, POWER.7, RESET.1, RESET.2, RN1.7, RN2.5, U1.1, U2.2, U3.3, U3.33, U5.4, X1.1, X1.3, Y2.2, ZU4.22, ZU4.8
- removed net IO0: IOL.1, RN4.2, ZU4.2
- removed net IO1: IOL.2, RN4.1, ZU4.3
- removed net IO2: IOL.3, ZU4.4
- removed net IO3: IOL.4, ZU4.5
- removed net IO4: IOL.5, ZU4.6
- removed net IO5: IOL.6, ZU4.11
- removed net IO6: IOL.7, ZU4.12
- removed net IO7: IOL.8, ZU4.13
- removed net IO8: IOH.1, ZU4.14
- removed net IO9: IOH.2, ZU4.15
- removed net L13: RN2.8, U5.6, U5.7
- removed net M8RXD: RN4.7, U3.9
- removed net M8TXD: RN4.8, U3.8
- removed net MISO: ICSP.1, IOH.5, ZU4.18
- removed net MISO2: ICSP1.1, U3.17
- removed net MOSI: ICSP.4, IOH.4, ZU4.17
- removed net MOSI2: ICSP1.4, U3.16
- removed net N$1: L.A, RN2.1
- removed net N$3: ON.A, RN4.5, RN4.6
- removed net N$35: RN2.7, RX.A
- removed net N$36: RN2.6, TX.A
- removed net PB4: JP2.1, U3.18
- removed net PB5: JP2.3, U3.19
- removed net PB6: JP2.2, U3.20
- removed net PB7: JP2.4, U3.21
- removed net PWRIN: D1.A, X1.2
- removed net RD+: RN3.4, U3.29
- removed net RD-: RN3.1, U3.30
- removed net RESET: C5.2, D2.A, ICSP.5, POWER.3, RESET-EN.1, RESET-EN.2, RESET.3, RESET.4, RN1.4, ZU4.1
- removed net RESET2: D3.A, ICSP1.5, RN1.6, U3.24
- removed net RXLED: RX.C, U3.10
- removed net SCK: ICSP.3, IOH.6, U5.5, ZU4.19
- removed net SCK2: ICSP1.3, U3.15
- removed net SS: IOH.3, ZU4.16
- removed net TP_VUCAP: C8.1, U3.27
- removed net TXLED: TX.C, U3.11
- removed net UGND: C8.2, GROUND.2, L1.1, U3.28, X2.4
- removed net USBVCC: F1.1, T1.1, U3.31
- removed net USHIELD: L1.2, X2.P$1, X2.P$2, Z1.2, Z2.2
- removed net VIN: D1.C, PC1.+, POWER.8, RN1.8, U1.3
- removed net XT1: C9.1, R1.1, U3.1, Y1.2
- removed net XT2: C11.1, R1.2, U3.2, Y1.1
- removed net XTAL1: R2.1, Y2.3, ZU4.9
- removed net XTAL2: R2.2, Y2.1, ZU4.10
- removed net XUSB: F1.2, X2.1
Routing:
- net +5V: track 219.6 -> 0.00 mm, vias 15 -> 0
- net RESET: track 141.0 -> 0.00 mm, vias 3 -> 0
- net SCK: track 106.6 -> 0.00 mm, vias 1 -> 0
- net MISO: track 96.7 -> 0.00 mm, vias 1 -> 0
- net MOSI: track 90.8 -> 0.00 mm, vias 1 -> 0
- net AD5/SCL: track 88.1 -> 0.00 mm, vias 3 -> 0
- net VIN: track 81.8 -> 0.00 mm, vias 2 -> 0
- net AD4/SDA: track 81.1 -> 0.00 mm, vias 3 -> 0
- net AREF: track 73.9 -> 0.00 mm, vias 1 -> 0
- net RESET2: track 56.6 -> 0.00 mm, vias 2 -> 0
- net IO0: track 45.6 -> 0.00 mm, vias 1 -> 0
- net IO9: track 45.3 -> 0.00 mm, vias 1 -> 0
- net SS: track 43.8 -> 0.00 mm, vias 1 -> 0
- net IO1: track 39.2 -> 0.00 mm, vias 1 -> 0
- net UGND: track 39.1 -> 0.00 mm
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- removed copper zone on layer 1, net +5V
- removed copper zone on layer 16, net +5V
- removed copper zone on layer 1, net GND
- removed copper zone on layer 16, net GND
Other:
- board outline removed
- board text removed: "#"
- board text removed: "0"
- board text removed: "1"
- board text removed: "10"
- board text removed: "11"
- board text removed: "12"
- board text removed: "13"
- board text removed: "2"
- board text removed: "2011-3-02"
- board text removed: "3"
- board text removed: "3V3"
- board text removed: "4"
- board text removed: "5"
- board text removed: "5V"
- board text removed: "6"
- board text removed: "7"
- board text removed: "8"
- board text removed: "9"
- board text removed: "A0"
- board text removed: "A1"
- board text removed: "A2"
- board text removed: "A3"
- board text removed: "A4"
- board text removed: "A5"
- board text removed: "ANALOG IN"
- board text removed: "AREF"
- board text removed: "ATMEGA328"
- board text removed: "Arduino"
- board text removed: "D.Cuartielles"
- board text removed: "D.Mellis"
- board text removed: "DIGITAL"
- board text removed: "Edition"
- board text removed: "G.Martino"
- board text removed: "GND"
- board text removed: "IOREF"
- board text removed: "ITALY"
- board text removed: "L"
- board text removed: "Limited"
- board text removed: "M.Banzi"
- board text removed: "MADE IN"
- board text removed: "ON"
- board text removed: "PC1"
- board text removed: "PC2"
- board text removed: "Prototype"
- board text removed: "RESET"
- board text removed: "RX"
- board text removed: "SCL"
- board text removed: "SDA"
- board text removed: "T.Igoe"
- board text removed: "TM"
- board text removed: "TX"
- board text removed: "UNO"
- board text removed: "Use of the Arduino name must be compliant with http://www.arduino.cc/en/Main/Policy"
- board text removed: "VIN"
- board text removed: "[#=PWM]"
- board text removed: "designed by"
- board text removed: "tinker it"
- board text removed: "www.arduino.cc"

Commit message: got board to populate
Parts:
- added AUDIO_AMP:AMP1: MC1458, El14_AudioServo:DIP8
- added AUDIO_AMP:C1: .1uF, capacitor-wima:C2.5-3
- added AUDIO_AMP:JP1: (no value), SparkFun-Connectors:STEREOJACK2.5MM_STEREOJACK2.5MM
- added AUDIO_AMP:R1: 1k, resistor:0204/5
- added POWER:JP1: M02PTH, SparkFun-Connectors:1X02
Connections:
- new net AUDIO_AMP:N$1: AUDIO_AMP:AMP1.2, AUDIO_AMP:R1.2
- new net AUDIO_AMP:N$2: AUDIO_AMP:C1.2, AUDIO_AMP:R1.1
- new net AUDIO_AMP:N$3: AUDIO_AMP:C1.1, AUDIO_AMP:JP1.TIP
- new net N$1: AUDIO_AMP:AMP1.4, AUDIO_AMP:JP1.RING1, POWER:JP1.1
- new net N$2: AUDIO_AMP:AMP1.8, POWER:JP1.2
Other:
- board outline added: 160 x 100 mm
- board text removed: "D:/SmartProjects/Snc/a4_bn_logo2.bmp"
